File: kicad/tiva_arm_board/transistor_board.sch (KiCad schematic (older format))
At the start: 16 parts, among them J1 Conn_01x10, Q1 Q_NIGBT_GCEC, Q2 Q_NIGBT_GCEC, Q3 MMBF170, Q4 MMBF170, U2 ESP32-cam, U3 LM7805_TO220

Commit message: corrected the transistors
Parts:
- removed Q1, Q2: Q_NIGBT_GCEC, symbol Device:Q_NIGBT_GCEC
- added Q1, Q2: MMBF170, Package_TO_SOT_SMD:TO-252-3_TabPin2, symbol transistor_board-rescue:MMBF170-Transistor_FET
- added U?: TM4C1230C3PM, Package_QFP:LQFP-64_10x10mm_P0.5mm, symbol MCU_Texas:TM4C1230C3PM
Connections:
- wire segments 107 -> 105
Other:
- note added: "TODO This may not match the transistor we use."
Changed lines of the file:
@@
 EELAYER 30 0
 EELAYER END
-$Descr A4 11693 8268
+$Descr A3 16535 11693
 encoding utf-8
 Sheet 1 1
@@
 Wire Wire Line
 	4000 3750 3650 3750
+$Comp
+L transistor_board-rescue:MMBF170-Transistor_FET Q2
+U 1 1 5F261E90
+P 9050 3250
+F 0 "Q2" H 9254 3296 50  0000 L CNN
+F 1 "MMBF170" H 9254 3205 50  0000 L CNN
+F 2 "Package_TO_SOT_SMD:TO-252-3_TabPin2" H 9250 3175 50  0001 L CIN
+F 3 "https://www.diodes.com/assets/Datasheets/ds30104.pdf" H 9050 3250 50  0001 L CNN
+	1    9050 3250
+	1    0    0    -1
+$EndComp
+$Comp
+L transistor_board-rescue:MMBF170-Transistor_FET Q1
+U 1 1 5F263B9D
+P 9050 4150
+F 0 "Q1" H 9254 4196 50  0000 L CNN
+F 1 "MMBF170" H 9254 4105 50  0000 L CNN
+F 2 "Package_TO_SOT_SMD:TO-252-3_TabPin2" H 9250 4075 50  0001 L CIN
+F 3 "https://www.diodes.com/assets/Datasheets/ds30104.pdf" H 9050 4150 50  0001 L CNN
+	1    9050 4150
+	1    0    0    -1
+$EndComp
 Wire Wire Line
 	5800 1250 5800 2450
@@
 Connection ~ 9350 2900
 Wire Wire Line
-	9350 2900 9250 2900
+	9350 2900 9150 2900
 Wire Wire Line
 	10100 1800 10450 1800
@@
 Wire Wire Line
 	5200 1300 5200 1250
-$Comp
-L Device:Q_NIGBT_GCEC Q1
-U 1 1 606B90B8
-P 9050 3250
-F 0 "Q1" H 9338 3296 50  0000 L CNN
-F 1 "Q_NIGBT_GCEC" H 9338 3205 50  0000 L CNN
-F 2 "" H 9250 3350 50  0001 C CNN
-F 3 "~" H 9050 3250 50  0001 C CNN
-	1    9050 3250
-	1    0    0    -1
-$EndComp
-Wire Wire Line
-	9250 3050 9250 2900
-Connection ~ 9250 2900
-Wire Wire Line
-	9250 2900 9150 2900
-$Comp
-L Device:Q_NIGBT_GCEC Q2
-U 1 1 606C00AA
-P 9050 4150
-F 0 "Q2" H 9338 4196 50  0000 L CNN
-F 1 "Q_NIGBT_GCEC" H 9338 4105 50  0000 L CNN
-F 2 "" H 9250 4250 50  0001 C CNN
-F 3 "~" H 9050 4150 50  0001 C CNN
-	1    9050 4150
-	1    0    0    -1
-$EndComp
+Text Notes 8800 3050 0    50   ~ 0
+TODO This may not match the transistor we use.
+$Comp
+L MCU_Texas:TM4C1230C3PM U?
+U 1 1 605BD082
+P 2750 6900
+F 0 "U?" H 2750 4811 50  0000 C CNN
+F 1 "TM4C1230C3PM" H 2750 4720 50  0000 C CNN
+F 2 "Package_QFP:LQFP-64_10x10mm_P0.5mm" H 4000 4900 50  0001 C CIN
+F 3 "http://www.ti.com/lit/ds/symlink/tm4c1230c3pm.pdf" H 2750 6900 50  0001 C CNN
+	1    2750 6900
+	1    0    0    -1
+$EndComp
