File: kicad/transistor_board/transistor_board.kicad_pcb (KiCad board)
At the start: 2 copper layers, 25.4 x 38.1 mm, 16 parts, among them J1 Conn_01x10, Q1 Q_NIGBT_GCEC, Q2 Q_NIGBT_GCEC, Q3 MMBF170, Q4 MMBF170, U2 ESP32-cam, U3 LM7805_TO220

Commit message: prepared files to send to JLCPCB for assembly
Parts:
- C3, C6: value C -> 10 uF; footprint Capacitor_SMD:C_0805_2012Metric_Pad1.15x1.40mm_HandSolder -> Capacitor_SMD:C_1206_3216Metric
- C5: value C -> 1 uF; footprint Capacitor_SMD:C_0805_2012Metric_Pad1.15x1.40mm_HandSolder -> Capacitor_SMD:C_0805_2012Metric
- Q1, Q2: value Q_NIGBT_GCEC -> Q_NIGBT_GCE
- R2: value R -> 10K; footprint Resistor_SMD:R_0805_2012Metric -> Resistor_SMD:R_0805_2012Metric_Pad1.15x1.40mm_HandSolder
- R3: value R -> 1K5; footprint Resistor_SMD:R_0805_2012Metric -> Resistor_SMD:R_0805_2012Metric_Pad1.15x1.40mm_HandSolder
- moved C3 1.39 mm to (128.4, 122.4), turned to 0 degrees
- moved Q2 0.09 mm to (120.4, 103.4)
- moved Q1 0.08 mm to (132.0, 103.4)
Connections:
- net Net-(C3-Pad1) renamed /Com
- net Net-(C6-Pad2) renamed /Cap+
- net Net-(D1-Pad3) renamed /AC1
- net Net-(D1-Pad4) renamed /AC2
- net Net-(D3-Pad1) renamed /Reverse
- net Net-(D3-Pad2) renamed /Forward
- net Net-(J1-Pad7) renamed /Lights_forward
- net Net-(J1-Pad8) renamed /Lights_reverse
- U2 pad 1: Net-(U2-Pad1) -> (no net)
- U2 pad 7: Net-(U2-Pad7) -> (no net)
Routing:
- net GND: track 78.7 -> 81.1 mm
- net /Com: track 56.4 -> 58.0 mm
